Commit message: save current urdf changes.

File: src/my_robot_description/xacro/camera.xacro (robot description, xacro)
@@ -28,26 +28,28 @@
     </joint>
     <link name="camera_link_optical"></link>
-    <gazebo reference="camera_link">
-        <material>Gazebo/Red</material>
-        <sensor name="camera" type="camera">
-            <pose>0 0 0 0 0 0</pose>
-            <visualize>true</visualize>
-            <update_rate>10</update_rate>
-            <camera>
-                <horizontal>1.089</horizontal>
-                <image>
-                    <format>R8G8B9</format>
-                    <width>640</width>
-                    <height>480</height>
-                </image>
-                <clip>
-                    <near>0.05</near>
-                    <far>8.0</far>
-                </clip>
-            </camera>
-            <plugin name="camera_controller" filename="libgazebo_ros_camera.so">
-                <frame_name>camera_link_optical</frame_name>
-            </plugin>
-        </sensor>
-    </gazebo>
+    <xacro:if value="$(arg sim_mode)">
+        <gazebo reference="camera_link">
+            <material>Gazebo/Red</material>
+            <sensor name="camera" type="camera">
+                <pose>0 0 0 0 0 0</pose>
+                <visualize>true</visualize>
+                <update_rate>10</update_rate>
+                <camera>
+                    <horizontal>1.089</horizontal>
+                    <image>
+                        <format>R8G8B9</format>
+                        <width>640</width>
+                        <height>480</height>
+                    </image>
+                    <clip>
+                        <near>0.05</near>
+                        <far>8.0</far>
+                    </clip>
+                </camera>
+                <plugin name="camera_controller" filename="libgazebo_ros_camera.so">
+                    <frame_name>camera_link_optical</frame_name>
+                </plugin>
+            </sensor>
+        </gazebo>
+    </xacro:if>
 </robot>

File: src/my_robot_description/xacro/gps.xacro (robot description, xacro)
@@ -30,15 +30,17 @@
         </sensor> -->
     </link>
-    <gazebo reference="gps_link">
-        <sensor name="gps_sensor" type="gps">
-            <always_on>true</always_on>
-            <update_rate>1.0</update_rate>
-            <plugin name="gps_controller" filename="libgazebo_ros_gps_sensor.so">
-                <ros>
-                    <remapping>~/out:=/gps/fix</remapping>
-                </ros>
-                <frame_name>gps_link</frame_name>
-            </plugin>
-        </sensor>
-    </gazebo>
+    <xacro:if value="$(arg sim_mode)">
+        <gazebo reference="gps_link">
+            <sensor name="gps_sensor" type="gps">
+                <always_on>true</always_on>
+                <update_rate>1.0</update_rate>
+                <plugin name="gps_controller" filename="libgazebo_ros_gps_sensor.so">
+                    <ros>
+                        <remapping>~/out:=/gps/fix</remapping>
+                    </ros>
+                    <frame_name>gps_link</frame_name>
+                </plugin>
+            </sensor>
+        </gazebo>
+    </xacro:if>
 </robot>

File: src/my_robot_description/xacro/imu.xacro (robot description, xacro)
@@ -8,16 +8,18 @@
     <link name="imu_link">
     </link>
-    <gazebo reference="imu_link">
-        <sensor name="imu_sensor" type="imu">
-            <always_on>true</always_on>
-            <update_rate>50</update_rate>
-            <plugin name="gazebo_ros_imu" filename="libgazebo_ros_imu_sensor.so">
-                <ros>
-                    <remapping>~/out:=/imu/data</remapping>
-                </ros>
-                <frame_name>imu_link</frame_name>
-                <gaussianNoise>0.0002</gaussianNoise>
-            </plugin>
-        </sensor>
-    </gazebo>
+    <xacro:if value="$(arg sim_mode)">
+        <gazebo reference="imu_link">
+            <sensor name="imu_sensor" type="imu">
+                <always_on>true</always_on>
+                <update_rate>50</update_rate>
+                <plugin name="gazebo_ros_imu" filename="libgazebo_ros_imu_sensor.so">
+                    <ros>
+                        <remapping>~/out:=/imu/data</remapping>
+                    </ros>
+                    <frame_name>imu_link</frame_name>
+                    <gaussianNoise>0.0002</gaussianNoise>
+                </plugin>
+            </sensor>
+        </gazebo>
+    </xacro:if>
 </robot>

File: src/my_robot_description/xacro/lidar.xacro (robot description, xacro)
@@ -22,35 +22,37 @@
         </xacro:inertial_cylinder>
     </link>
-    <gazebo reference="lidar_frame">
-        <material>Gazebo/Red</material>
-        <sensor name="lidar" type="ray">
-            <pose>0 0 0 0 0 0</pose>
-            <visualize>true</visualize>
-            <update_rate>10</update_rate>
-            <ray>
-                <scan>
-                    <horizontal>
-                        <samples>360</samples>
-                        <resolution>1</resolution>
-                        <min_angle>-3.14</min_angle>
-                        <max_angle>3.14</max_angle>
-                    </horizontal>
-                </scan>
-                <range>
-                    <min>0.3</min>
-                    <max>30.0</max>
-                    <resolution>0.01</resolution>
-                </range>
-            </ray>
-            <plugin name="lidar_controller" filename="libgazebo_ros_ray_sensor.so">
-                <ros>
-                    <argument>
-                        ~/out:=scan
-                    </argument>
-                </ros>
-                <output_type>sensor_msgs/LaserScan</output_type>
-                <frame_name>lidar_frame</frame_name>
-            </plugin>
-        </sensor>
-    </gazebo>
+    <xacro:if value="$(arg sim_mode)">
+        <gazebo reference="lidar_frame">
+            <material>Gazebo/Red</material>
+            <sensor name="lidar" type="ray">
+                <pose>0 0 0 0 0 0</pose>
+                <visualize>true</visualize>
+                <update_rate>10</update_rate>
+                <ray>
+                    <scan>
+                        <horizontal>
+                            <samples>360</samples>
+                            <resolution>1</resolution>
+                            <min_angle>-3.14</min_angle>
+                            <max_angle>3.14</max_angle>
+                        </horizontal>
+                    </scan>
+                    <range>
+                        <min>0.3</min>
+                        <max>30.0</max>
+                        <resolution>0.01</resolution>
+                    </range>
+                </ray>
+                <plugin name="lidar_controller" filename="libgazebo_ros_ray_sensor.so">
+                    <ros>
+                        <argument>
+                            ~/out:=scan
+                        </argument>
+                    </ros>
+                    <output_type>sensor_msgs/LaserScan</output_type>
+                    <frame_name>lidar_frame</frame_name>
+                </plugin>
+            </sensor>
+        </gazebo>
+    </xacro:if>
 </robot>

File: src/my_robot_description/xacro/lidar_3d.xacro (robot description, xacro)
@@ -22,41 +22,43 @@
         </xacro:inertial_cylinder>
     </link>
-    <gazebo reference="lidar_frame">
-        <material>Gazebo/Red</material>
-        <sensor name="lidar" type="gpu_ray">
-            <pose>0 0 0 0 0 0</pose>
-            <visualize>true</visualize>
-            <update_rate>10</update_rate>
-            <ray>
-                <scan>
-                    <horizontal>
-                        <samples>1024</samples>             <!-- Horizontal Angular resolution -->
-                        <resolution>1</resolution>
-                        <min_angle>-3.14</min_angle>
-                        <max_angle>3.14</max_angle>
-                    </horizontal>
-                    <vertical>
-                        <samples>16</samples>               <!-- Vertical Beam Multilayer -->
-                        <min_angle>-0.2</min_angle>
-                        <max_angle>0.1</max_angle>
-                    </vertical>
-                </scan>
-                <range>
-                    <min>0.3</min>
-                    <max>10.0</max>
-                    <resolution>0.01</resolution>
-                </range>
-            </ray>
-            <plugin name="lidar_controller" filename="libgazebo_ros_ray_sensor.so">
-                <ros>
-                    <argument>
-                        ~/out:=points
-                    </argument>
-                </ros>
-                <output_type>sensor_msgs/PointCloud2</output_type>
-                <frame_name>lidar_frame</frame_name>
-                <use_sim_time>true</use_sim_time>
-            </plugin>
-        </sensor>
-    </gazebo>
+    <xacro:if value="$(arg sim_mode)">
+        <gazebo reference="lidar_frame">
+            <material>Gazebo/Red</material>
+            <sensor name="lidar" type="gpu_ray">
+                <pose>0 0 0 0 0 0</pose>
+                <visualize>true</visualize>
+                <update_rate>10</update_rate>
+                <ray>
+                    <scan>
+                        <horizontal>
+                            <samples>1024</samples>             <!-- Horizontal Angular resolution -->
+                            <resolution>1</resolution>
+                            <min_angle>-3.14</min_angle>
+                            <max_angle>3.14</max_angle>
+                        </horizontal>
+                        <vertical>
+                            <samples>16</samples>               <!-- Vertical Beam Multilayer -->
+                            <min_angle>-0.2</min_angle>
+                            <max_angle>0.1</max_angle>
+                        </vertical>
+                    </scan>
+                    <range>
+                        <min>0.3</min>
+                        <max>10.0</max>
+                        <resolution>0.01</resolution>
+                    </range>
+                </ray>
+                <plugin name="lidar_controller" filename="libgazebo_ros_ray_sensor.so">
+                    <ros>
+                        <argument>
+                            ~/out:=points
+                        </argument>
+                    </ros>
+                    <output_type>sensor_msgs/PointCloud2</output_type>
+                    <frame_name>lidar_frame</frame_name>
+                    <use_sim_time>true</use_sim_time>
+                </plugin>
+            </sensor>
+        </gazebo>
+    </xacro:if>
 </robot>

File: src/my_robot_description/xacro/robot.urdf.xacro (robot description, xacro)
@@ -2,4 +2,5 @@
 <robot xmlns:xacro="http://www.ros.org/wiki/xacro"  name="robot">
     <xacro:arg name="use_ros2_control" default="true"/>
+    <xacro:arg name="sim_mode" default="false"/>
     <xacro:include filename="robot_core.xacro"/>
     <xacro:if value="$(arg use_ros2_control)">

File: src/my_robot_description/xacro/robot_core.xacro (robot description, xacro)
@@ -42,21 +42,46 @@
     <link name="chassis">
         <visual>
-            <origin xyz="0.45 0 0.35" />
+            <origin xyz="0.45 0 0.1" />
             <geometry>
-                <box size="0.9 0.7 0.7"/>
+                <box size="0.9 0.4 0.2"/>
             </geometry>
             <material name="white"/>
         </visual>
         <collision>
-            <origin xyz="0.45 0 0.35" />
+            <origin xyz="0.45 0 0.1" />
             <geometry>
-                <box size="0.9 0.7 0.7"/>
+                <box size="0.9 0.4 0.2"/>
             </geometry>
         </collision>
-        <xacro:inertial_box mass="0.5" x="0.9" y="0.5" z="0.7">
-            <origin xyz="0.45 0 0.35" rpy="0 0 0"/>
+        <xacro:inertial_box mass="0.5" x="0.9" y="0.4" z="0.2">
+            <origin xyz="0.45 0 0.1" rpy="0 0 0"/>
         </xacro:inertial_box>
     </link>
     <gazebo reference="chassis">
+        <material>Gazebo/White</material>
+    </gazebo>
+    <!-- SENSOR POLE -->
+    <joint name="pole_joint" type="fixed">
+    	<parent link="chassis"/>
+    	<child link="pole"/>
+    	<origin xyz="0.45 0 0.4"/>
+    </joint>
+    <link name="pole">
+    	<visual>
+    	    <geometry>
+    	    	<cylinder radius="0.03" length="0.6"/>
+    	    </geometry>
+    	    <material name="white"/>
+    	</visual>
+    	<collision>
+	   <geometry>
+    	    	<cylinder radius="0.03" length="0.6"/>
+    	    </geometry>
+    	</collision>
+    	<xacro:inertial_cylinder mass="0.2" length="0.6" radius="0.03">
+            <origin xyz="0 0 0" rpy="0 0 0"/>
+        </xacro:inertial_cylinder>
+    </link>
+    <gazebo reference="pole">
         <material>Gazebo/White</material>
     </gazebo>
@@ -65,5 +90,5 @@
         <parent link="base_link"/>
         <child link="left_wheel"/>
-        <origin xyz="0 0.35 0" rpy="-${pi/2} 0 0"/>
+        <origin xyz="0 0.4 0" rpy="-${pi/2} 0 0"/>
         <axis xyz="0 0 1"/>
     </joint>
@@ -71,5 +96,5 @@
         <visual>
             <geometry>
-                <cylinder radius="0.25" length="0.04"/>
+                <cylinder radius="0.125" length="0.086"/>
             </geometry>
             <material name="blue"/>
@@ -77,8 +102,8 @@
         <collision>
             <geometry>
-                <cylinder radius="0.25" length="0.04"/>
+                <cylinder radius="0.125" length="0.086"/>
             </geometry>
         </collision>
-        <xacro:inertial_cylinder mass="0.1" length="0.04" radius="0.25">
+        <xacro:inertial_cylinder mass="0.1" length="0.086" radius="0.125">
             <origin xyz="0 0 0" rpy="0 0 0"/>
         </xacro:inertial_cylinder>
@@ -91,5 +116,5 @@
         <parent link="base_link"/>
         <child link="right_wheel"/>
-        <origin xyz="0 -0.35 0" rpy="${pi/2} 0 0"/>
+        <origin xyz="0 -0.4 0" rpy="${pi/2} 0 0"/>
         <axis xyz="0 0 -1"/>
     </joint>
@@ -97,5 +122,5 @@
         <visual>
             <geometry>
-                <cylinder radius="0.25" length="0.04"/>
+                <cylinder radius="0.125" length="0.086"/>
             </geometry>
             <material name="blue"/>
@@ -103,8 +128,8 @@
         <collision>
             <geometry>
-                <cylinder radius="0.25" length="0.04"/>
+                <cylinder radius="0.125" length="0.086"/>
             </geometry>
         </collision>
-        <xacro:inertial_cylinder mass="0.1" length="0.04" radius="0.25">
+        <xacro:inertial_cylinder mass="0.1" length="0.086" radius="0.125">
             <origin xyz="0 0 0" rpy="0 0 0"/>
         </xacro:inertial_cylinder>
@@ -122,5 +147,5 @@
         <visual>
             <geometry>
-                <sphere radius="0.25"/>
+                <sphere radius="0.125"/>
             </geometry>
             <material name="black"/>
@@ -128,8 +153,8 @@
         <collision>
             <geometry>
-                <sphere radius="0.25"/>
+                <sphere radius="0.125"/>
             </geometry>
         </collision>
-        <xacro:inertial_sphere mass="0.1" radius="0.25">
+        <xacro:inertial_sphere mass="0.1" radius="0.125">
             <origin xyz="0 0 0" rpy="0 0 0"/>
         </xacro:inertial_sphere>
@@ -149,5 +174,5 @@
         <visual>
             <geometry>
-                <sphere radius="0.25"/>
+                <sphere radius="0.125"/>
             </geometry>
             <material name="black"/>
@@ -155,8 +180,8 @@
         <collision>
             <geometry>
-                <sphere radius="0.25"/>
+                <sphere radius="0.125"/>
             </geometry>
         </collision>
-        <xacro:inertial_sphere mass="0.1" radius="0.25">
+        <xacro:inertial_sphere mass="0.1" radius="0.125">
             <origin xyz="0 0 0" rpy="0 0 0"/>
         </xacro:inertial_sphere>

File: src/my_robot_description/xacro/ros2_control.xacro (robot description, xacro)
@@ -1,31 +1,56 @@
 <?xml version="1.0"?>
 <robot xmlns:xacro="http://www.ros.org/wiki/xacro">
-    <ros2_control name="GazeboSystem" type="system">
-        <hardware>
-            <plugin>gazebo_ros2_control/GazeboSystem</plugin>
-        </hardware>
-        <joint name="left_wheel_joint">
-            <command_interface name="velocity">
-                <param name="min">-10</param>
-                <param name="max">10</param>
-            </command_interface>
-            <state_interface name="velocity"/>
-            <state_interface name="position"/>
-        </joint>
-        <joint name="right_wheel_joint">
-            <command_interface name="velocity">
-                <param name="min">-10</param>
-                <param name="max">10</param>
-            </command_interface>
-            <state_interface name="velocity"/>
-            <state_interface name="position"/>
-        </joint>
-    </ros2_control>
-    <gazebo>
-        <plugin name="gazebo_ros2_control" filename="libgazebo_ros2_control.so">
-            <parameters>
-                $(find igvc_bot_description)/config/controllers.yaml
-            </parameters>
-        </plugin>
-    </gazebo>
+    <xacro:if value="$(arg sim_mode)">
+        <ros2_control name="GazeboSystem" type="system">
+            <hardware>
+                <plugin>gazebo_ros2_control/GazeboSystem</plugin>
+            </hardware>
+            <joint name="left_wheel_joint">
+                <command_interface name="velocity">
+                    <param name="min">-10</param>
+                    <param name="max">10</param>
+                </command_interface>
+                <state_interface name="velocity"/>
+                <state_interface name="position"/>
+            </joint>
+            <joint name="right_wheel_joint">
+                <command_interface name="velocity">
+                    <param name="min">-10</param>
+                    <param name="max">10</param>
+                </command_interface>
+                <state_interface name="velocity"/>
+                <state_interface name="position"/>
+            </joint>
+        </ros2_control>
+        <gazebo>
+            <plugin name="gazebo_ros2_control" filename="libgazebo_ros2_control.so">
+                <parameters>
+                    $(find my_robot_gazebo)/config/controllers.yaml
+                </parameters>
+            </plugin>
+        </gazebo>
+    </xacro:if>
+    <xacro:unless value="$(arg sim_mode)">
+        <ros2_control name="HardwareSystem" type="system">
+            <hardware>
+                <plugin></plugin>
+            </hardware>
+            <joint name="left_wheel_joint">
+                <command_interface name="velocity">
+                    <param name="min">-10</param>
+                    <param name="max">10</param>
+                </command_interface>
+                <state_interface name="velocity"/>
+                <state_interface name="position"/>
+            </joint>
+            <joint name="right_wheel_joint">
+                <command_interface name="velocity">
+                    <param name="min">-10</param>
+                    <param name="max">10</param>
+                </command_interface>
+                <state_interface name="velocity"/>
+                <state_interface name="position"/>
+            </joint>
+        </ros2_control>
+    </xacro:unless>
 </robot>
