Commit message: add hardware interface

File: src/my_robot_description/xacro/camera.xacro (robot description, xacro)
@@ -4,5 +4,5 @@
         <parent link="chassis"/>
         <child link="camera_link"/>
-        <origin xyz="0.905 0 0.4" rpy="0 0 0"/>
+        <origin xyz="0.4 0 0.65" rpy="0 0 0"/>
     </joint>
     <link name="camera_link">

File: src/my_robot_description/xacro/lidar_3d.xacro (robot description, xacro)
@@ -4,5 +4,5 @@
         <parent link="chassis"/>
         <child link="lidar_frame"/>
-        <origin xyz="0.45 0 0.71" rpy="0 0 0"/>
+        <origin xyz="0.305 0 0.71" rpy="0 0 0"/>
     </joint>
     <link name="lidar_frame">

File: src/my_robot_description/xacro/robot_core.xacro (robot description, xacro)
@@ -38,22 +38,22 @@
         <parent link="base_link"/>
         <child link="chassis"/>
-        <origin xyz="-0.45 0 0"/>
+        <origin xyz="-0.305 0 0"/>
     </joint>
     <link name="chassis">
         <visual>
-            <origin xyz="0.45 0 0.1" />
+            <origin xyz="0.305 0 0.1" />
             <geometry>
-                <box size="0.9 0.4 0.2"/>
+                <box size="0.61 0.455 0.2"/>
             </geometry>
             <material name="white"/>
         </visual>
         <collision>
-            <origin xyz="0.45 0 0.1" />
+            <origin xyz="0.305 0 0.1" />
             <geometry>
-                <box size="0.9 0.4 0.2"/>
+                <box size="0.61 0.455 0.2"/>
             </geometry>
         </collision>
-        <xacro:inertial_box mass="0.5" x="0.9" y="0.4" z="0.2">
-            <origin xyz="0.45 0 0.1" rpy="0 0 0"/>
+        <xacro:inertial_box mass="0.5" x="0.61" y="0.455" z="0.2">
+            <origin xyz="0.305 0 0.1" rpy="0 0 0"/>
         </xacro:inertial_box>
     </link>
@@ -65,5 +65,5 @@
     	<parent link="chassis"/>
     	<child link="pole"/>
-    	<origin xyz="0.45 0 0.4"/>
+    	<origin xyz="0.305 0 0.4"/>
     </joint>
     <link name="pole">
@@ -90,5 +90,5 @@
         <parent link="base_link"/>
         <child link="left_wheel"/>
-        <origin xyz="0 0.4 0" rpy="-${pi/2} 0 0"/>
+        <origin xyz="0 0.2705 0" rpy="-${pi/2} 0 0"/>
         <axis xyz="0 0 1"/>
     </joint>
@@ -96,5 +96,5 @@
         <visual>
             <geometry>
-                <cylinder radius="0.125" length="0.086"/>
+                <cylinder radius="0.128" length="0.085"/>
             </geometry>
             <material name="blue"/>
@@ -102,8 +102,8 @@
         <collision>
             <geometry>
-                <cylinder radius="0.125" length="0.086"/>
+                <cylinder radius="0.128" length="0.085"/>
             </geometry>
         </collision>
-        <xacro:inertial_cylinder mass="0.1" length="0.086" radius="0.125">
+        <xacro:inertial_cylinder mass="0.1" length="0.085" radius="0.128">
             <origin xyz="0 0 0" rpy="0 0 0"/>
         </xacro:inertial_cylinder>
@@ -116,5 +116,5 @@
         <parent link="base_link"/>
         <child link="right_wheel"/>
-        <origin xyz="0 -0.4 0" rpy="${pi/2} 0 0"/>
+        <origin xyz="0 -0.2705 0" rpy="${pi/2} 0 0"/>
         <axis xyz="0 0 -1"/>
     </joint>
@@ -122,5 +122,5 @@
         <visual>
             <geometry>
-                <cylinder radius="0.125" length="0.086"/>
+                <cylinder radius="0.128" length="0.085"/>
             </geometry>
             <material name="blue"/>
@@ -128,8 +128,8 @@
         <collision>
             <geometry>
-                <cylinder radius="0.125" length="0.086"/>
+                <cylinder radius="0.128" length="0.085"/>
             </geometry>
         </collision>
-        <xacro:inertial_cylinder mass="0.1" length="0.086" radius="0.125">
+        <xacro:inertial_cylinder mass="0.1" length="0.085" radius="0.128">
             <origin xyz="0 0 0" rpy="0 0 0"/>
         </xacro:inertial_cylinder>
@@ -142,5 +142,5 @@
         <parent link="chassis"/>
         <child link="caster_wheel_front"/>
-        <origin xyz="0.89 0 0"/>
+        <origin xyz="0.6 0 0"/>
     </joint>
     <link name="caster_wheel_front">

File: src/my_robot_description/xacro/ros2_control.xacro (robot description, xacro)
@@ -8,6 +8,6 @@
             <joint name="left_wheel_joint">
                 <command_interface name="velocity">
-                    <param name="min">-10</param>
-                    <param name="max">10</param>
+                    <param name="min">-8.047</param>
+                    <param name="max">8.047</param>
                 </command_interface>
                 <state_interface name="velocity"/>
@@ -16,6 +16,6 @@
             <joint name="right_wheel_joint">
                 <command_interface name="velocity">
-                    <param name="min">-10</param>
-                    <param name="max">10</param>
+                    <param name="min">-8.047</param>
+                    <param name="max">8.047</param>
                 </command_interface>
                 <state_interface name="velocity"/>
@@ -34,10 +34,19 @@
         <ros2_control name="HardwareSystem" type="system">
             <hardware>
-                <plugin></plugin>
+                <plugin>my_robot_description/DiffDriveArduinoHardware</plugin>
+                <param name="left_wheel_name">left_wheel_joint</param>
+                <param name="loop_rate">50</param>
+                <param name="right_wheel_name">right_wheel_joint</param>
+                <!-- device port subject to change -->
+                <param name="device">/dev/serial/by-path/platform-fd500000.pcie-pci-0000:01:00.0-usb-0:1.3:1.0-port0</param>
+                <param name="baud_rate">115200</param>
+                <param name="timeout_ms">1000</param>
+                <param name="enc_counts_per_rev">9650</param>
+                <!-- <param name="pid_o">50</param> -->
             </hardware>
             <joint name="left_wheel_joint">
                 <command_interface name="velocity">
-                    <param name="min">-10</param>
-                    <param name="max">10</param>
+                    <param name="min">-8.047</param>
+                    <param name="max">8.047</param>
                 </command_interface>
                 <state_interface name="velocity"/>
@@ -46,6 +55,6 @@
             <joint name="right_wheel_joint">
                 <command_interface name="velocity">
-                    <param name="min">-10</param>
-                    <param name="max">10</param>
+                    <param name="min">-8.047</param>
+                    <param name="max">8.047</param>
                 </command_interface>
                 <state_interface name="velocity"/>
